File: raspi_hat.kicad_pcb (KiCad board)
At the start: 2 copper layers, 69.9 x 56 mm, 5 parts, among them J1 Raspberry_Pi_2_3, Q1 BSS138, Q2 BSS138, U1 ATtiny85-20SU, U2 74LVC1G97

Commit message: add power parts
Parts:
- added IC1: DMMT5401-7-F, DMMT5401-7-F:DMMT5401-7-F, F.Cu at (74.9, 82.5)
- added J3: 39502-1003, 39502-1003:39502-1003, B.Cu at (63.0, 98.0)
- added L1: SRU1048-150Y, SRU1048-150Y:SRU1048-150Y, F.Cu at (64.8, 81.3)
- added PS1: TPS54202DDCR, TPS54202DDCR:TPS54202DDCR, F.Cu at (75.0, 76.2)
- added Q3: DMG2305UX-7, DMG2305UX-7:DMG2305UX-7, F.Cu at (74.9, 69.8)
- added R1: R, Resistor_SMD:R_0805_2012Metric_Pad1.20x1.40mm_HandSolder, F.Cu at (95.2, 73.4)
- added R2: R, Resistor_SMD:R_0805_2012Metric_Pad1.20x1.40mm_HandSolder, F.Cu at (87.4, 66.0)
- moved U2 29.0 mm to (80.0, 96.5)
- moved Q1 19.8 mm to (85.1, 72.4)
- moved Q2 19.2 mm to (90.2, 72.4)
- moved U1 8.52 mm to (85.1, 85.1), turned to 90 degrees
Connections:
- J1 pad 10: Net-(J1-Pad10) -> RPI_RXD
- J1 pad 12: Net-(J1-Pad12) -> LED_STRIP_1
- J1 pad 35: Net-(J1-Pad35) -> LED_STRIP_2
- J1 pad 8: Net-(J1-Pad8) -> RPI_TXD
- U1 pad 2: Net-(U1-Pad2) -> LED_STRIP_1
- U1 pad 3: Net-(U1-Pad3) -> LED_STRIP_2
- U1 pad 4: Net-(U1-Pad4) -> GND
- U1 pad 5: Net-(U1-Pad5) -> RPI_TXD
- U1 pad 6: Net-(U1-Pad6) -> RPI_RXD
- U1 pad 8: Net-(U1-Pad8) -> +5V
Other:
- board size 69.9 x 56 mm -> 65 x 56 mm
- board text added: "https://hu.farnell.com/molex/39502-1003/terminal-block-header-3pos-th/dp/3222075 https://hu.farnell.com/molex/39500-0003/terminal-block-pluggable-3way/dp/3863555?ost=39500-0003"
- board text added: "rpi pos x 90 y 60"

Commit message: power save
Parts:
- added C1: 10uF/50V, Capacitor_SMD:C_1206_3216Metric_Pad1.33x1.80mm_HandSolder, F.Cu at (109.2, 77.5)
- added C2: 10uF/50V, Capacitor_SMD:C_1206_3216Metric_Pad1.33x1.80mm_HandSolder, F.Cu at (109.2, 81.3)
- added C3: 100nF/50V, Capacitor_SMD:C_0603_1608Metric_Pad1.08x0.95mm_HandSolder, F.Cu at (105.4, 68.6)
- added C4: 91pF, Capacitor_SMD:C_0603_1608Metric_Pad1.08x0.95mm_HandSolder, F.Cu at (120.7, 67.7)
- added C5: 22uF, Capacitor_SMD:C_1206_3216Metric_Pad1.33x1.80mm_HandSolder, F.Cu at (96.8, 66.0)
- added C6: 22uF, Capacitor_SMD:C_1206_3216Metric_Pad1.33x1.80mm_HandSolder, F.Cu at (96.8, 69.8)
- added C7: 22uF, Capacitor_SMD:C_1206_3216Metric_Pad1.33x1.80mm_HandSolder, F.Cu at (96.8, 73.7)
- added J4: Jack-DC, Connector_BarrelJack:BarrelJack_Horizontal, B.Cu at (68.6, 101.6)
- added R3: 100k, Resistor_SMD:R_0603_1608Metric_Pad0.98x0.95mm_HandSolder, F.Cu at (114.3, 73.3)
- added R4: 100k, Resistor_SMD:R_0603_1608Metric_Pad0.98x0.95mm_HandSolder, F.Cu at (116.8, 67.3)
- added R5: 13.7k, Resistor_SMD:R_0603_1608Metric_Pad0.98x0.95mm_HandSolder, F.Cu at (114.3, 67.3)
- added R6: 10k, Resistor_SMD:R_0805_2012Metric_Pad1.20x1.40mm_HandSolder, F.Cu at (84.8, 69.8)
- added R7: 47k, Resistor_SMD:R_0805_2012Metric_Pad1.20x1.40mm_HandSolder, F.Cu at (85.1, 66.0)
- added U3: 74LVC1G97, Package_TO_SOT_SMD:SOT-363_SC-70-6_Handsoldering, F.Cu at (81.3, 81.3)
- R1, R2: value R -> 10k
- moved PS1 34.9 mm to (109.2, 69.8), turned to 90 degrees
- moved J3 33.2 mm to (63.0, 64.8)
- moved L1 31.8 mm to (96.5, 82.5), turned to 180 degrees
- moved U1 21.6 mm to (63.5, 83.8)
- moved Q2 21.4 mm to (70.1, 80.0)
- moved R1 21.3 mm to (76.2, 82.8)
- moved Q1 19.8 mm to (71.1, 86.4)
- moved R2 17.6 mm to (75.2, 78.7)
- moved IC1 16.7 mm to (77.5, 66.0), turned to 180 degrees
- moved U2 8.98 mm to (81.3, 87.6)
- moved Q3 5.39 mm to (71.1, 66.0), turned to 270 degrees
Connections:
- net RPI_TXD renamed ATTINY_RX
- IC1 pad 2: Net-(IC1-Pad2) -> Net-(IC1-Pad1)
- IC1 pad 3: Net-(IC1-Pad3) -> Net-(IC1-Pad1)
- IC1 pad 5: Net-(IC1-Pad5) -> 5V_RPI
- IC1 pad 6: Net-(IC1-Pad6) -> +5V
- J1 pad 14: Net-(J1-Pad14) -> GND
- J1 pad 2: Net-(J1-Pad2) -> 5V_RPI
- J1 pad 20: Net-(J1-Pad20) -> GND
- J1 pad 25: Net-(J1-Pad25) -> GND
- J1 pad 30: Net-(J1-Pad30) -> GND
- J1 pad 34: Net-(J1-Pad34) -> GND
- J1 pad 39: Net-(J1-Pad39) -> GND
- J1 pad 4: Net-(J1-Pad4) -> 5V_RPI
- J1 pad 6: Net-(J1-Pad6) -> GND
- J1 pad 9: Net-(J1-Pad9) -> GND
- L1 pad 1: Net-(L1-Pad1) -> Net-(C3-Pad2)
- L1 pad 2: Net-(L1-Pad2) -> +5V
- PS1 pad 1: Net-(PS1-Pad1) -> GND
- PS1 pad 2: Net-(PS1-Pad2) -> Net-(C3-Pad2)
- PS1 pad 3: Net-(PS1-Pad3) -> VIN
- Q2 pad 2: LV -> RPI_RXD
- Q2 pad 3: HV -> ATTINY_TX
- Q3 pad 1: Net-(Q3-Pad1) -> Net-(IC1-Pad4)
- Q3 pad 2: Net-(Q3-Pad2) -> 5V_RPI
- Q3 pad 3: Net-(Q3-Pad3) -> +5V
- R1 pad 2: LV -> RPI_RXD
- R2 pad 2: HV -> ATTINY_TX
- U1 pad 6: RPI_RXD -> ATTINY_TX

Commit message: big save before Pico
Parts:
- removed C7: 22uF, Capacitor_SMD:C_1206_3216Metric_Pad1.33x1.80mm_HandSolder
- added IC2: MC74HC32ADG, MC74HC32ADG:MC74HC32ADG, B.Cu at (78.7, 85.1)
- added J2: Conn_02x20_Counter_Clockwise, Connector_PinHeader_2.54mm:PinHeader_2x20_P2.54mm_Vertical, F.Cu at (148.6, 115.6)
- added J5: 39502-1003, 39502-1003:39502-1003, F.Cu at (7.62, 96.5)
- added J6: 39502-1002, 39502-1002:39502-1002, F.Cu at (63.5, 66.0)
- added J7: 39502-1002, 39502-1002:39502-1002, F.Cu at (63.5, 100.3)
- added R10: 10k, Resistor_SMD:R_0805_2012Metric_Pad1.20x1.40mm_HandSolder, F.Cu at (44.9, 97.0)
- added R11: 10k, Resistor_SMD:R_0805_2012Metric_Pad1.20x1.40mm_HandSolder, F.Cu at (44.9, 99.9)
- added R8: ?, Resistor_SMD:R_0603_1608Metric_Pad0.98x0.95mm_HandSolder, F.Cu at (224.8, 113.0)
- added R9: 13.3k, Resistor_SMD:R_0603_1608Metric_Pad0.98x0.95mm_HandSolder, F.Cu at (228.6, 112.1)
- added U4: SC0915, raspberry-pi-pico-r3-1:raspberry-pi-pico-r3-1, F.Cu at (82.5, 85.1)
- C4: value 91pF -> 75pF
- J3, J4: moved to F.Cu
- R3: value 100k -> ?
- R4: value 100k -> 49.9k
- R5: value 13.7k -> 100k
- moved C3 123.3 mm to (223.5, 104.1), turned to 180 degrees
- moved R5 121.3 mm to (228.6, 108.0)
- moved PS1 118.1 mm to (221.0, 108.0), turned to 0 degrees
- moved R4 117.3 mm to (228.6, 102.9), turned to 90 degrees
- moved C6 117.1 mm to (209.8, 100.3)
- moved C5 116.7 mm to (209.8, 95.2)
- moved IC1 113.4 mm to (186.7, 96.5)
- moved Q3 113.4 mm to (180.3, 96.5)
- moved R3 113.0 mm to (220.1, 113.0), turned to 180 degrees
- moved C4 113.0 mm to (226.1, 108.4)
- moved R6 111.8 mm to (192.8, 99.1)
- moved R7 111.6 mm to (192.8, 95.2)
- moved C1 109.8 mm to (214.6, 108.2), turned to 90 degrees
- moved L1 107.1 mm to (201.9, 101.6), turned to 90 degrees
- moved C2 103.9 mm to (209.6, 108.2), turned to 90 degrees
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Connections:
- C4 pad 2: +5V -> Net-(C4-Pad2)
- PS1 pad 4: Net-(C4-Pad1) -> Net-(C4-Pad2)
- Q1 pad 1: Net-(Q1-Pad1) -> +3V3
- Q1 pad 2: Net-(Q1-Pad2) -> RPI_RXD
- Q1 pad 3: Net-(Q1-Pad3) -> ATTINY_TX
- R5 pad 1: GND -> Net-(C4-Pad2)
Other:
- board text added: "itt lehetne a táp"
- board text added: "octopart: gdhFT445!!%"
