File: raspi_hat.sch (KiCad schematic (older format))
At the start: 8 parts, among them J1 Raspberry_Pi_2_3, J2 Conn_02x20_Counter_Clockwise, Q1 BSS138, Q2 BSS138, U1 ATtiny85-20SU, U2 74LVC1G97

Commit message: add power parts
Parts:
- added IC1: DMMT5401-7-F, DMMT5401-7-F:DMMT5401-7-F, symbol DMMT5401-7-F:DMMT5401-7-F
- added J3: 39502-1003, 39502-1003:39502-1003, symbol 39502-1003:39502-1003
- added L1: SRU1048-150Y, SRU1048-150Y:SRU1048-150Y, symbol SRU1048-150Y:SRU1048-150Y
- added PS1: TPS54202DDCR, TPS54202DDCR:TPS54202DDCR, symbol TPS54202DDCR:TPS54202DDCR
- added Q3: DMG2305UX-7, DMG2305UX-7:DMG2305UX-7, symbol DMG2305UX-7:DMG2305UX-7
- R1, R2: footprint (none) -> Resistor_SMD:R_0805_2012Metric_Pad1.20x1.40mm_HandSolder
Connections:
- net +5V: now also U1.8 (VCC)
- net GND: now also U1.4 (GND)
- net RPI_RXD: now reaches J1.10 (GPIO15/RXD)
- net RPI_RXD: now also U1.6 (PB1)
- net LED_STRIP_1: now reaches J1.12 (GPIO18/PWM0)
- net LED_STRIP_1: now also U1.2 (XTAL1/PB3)
- net LED_STRIP_2: now reaches J1.35 (GPIO19/MISO1)
- net LED_STRIP_2: now also U1.3 (XTAL2/PB4)
- net RPI_TXD: now reaches J1.8 (GPIO14/TXD)
- net RPI_TXD: now also U1.5 (AREF/PB0)
Other:
- note added: "nem végleges, csak, hogy lássam a légvezetékeket"
- moved on the sheet: J1, Q2, R1, R2, U1, U2

Commit message: power save
Parts:
- added C1, C2: 10uF/50V, Capacitor_SMD:C_1206_3216Metric_Pad1.33x1.80mm_HandSolder, symbol Device:C
- added C3: 100nF/50V, Capacitor_SMD:C_0603_1608Metric_Pad1.08x0.95mm_HandSolder, symbol Device:C
- added C4: 91pF, Capacitor_SMD:C_0603_1608Metric_Pad1.08x0.95mm_HandSolder, symbol Device:C
- added C5, C6, C7: 22uF, Capacitor_SMD:C_1206_3216Metric_Pad1.33x1.80mm_HandSolder, symbol Device:CP
- added J4: Jack-DC, Connector_BarrelJack:BarrelJack_Horizontal, symbol Connector:Jack-DC
- added R3, R4: 100k, Resistor_SMD:R_0603_1608Metric_Pad0.98x0.95mm_HandSolder, symbol Device:R
- added R5: 13.7k, Resistor_SMD:R_0603_1608Metric_Pad0.98x0.95mm_HandSolder, symbol Device:R
- added R6: 10k, Resistor_SMD:R_0805_2012Metric_Pad1.20x1.40mm_HandSolder, symbol Device:R
- added R7: 47k, Resistor_SMD:R_0805_2012Metric_Pad1.20x1.40mm_HandSolder, symbol Device:R
- added U3: 74LVC1G97, Package_TO_SOT_SMD:SOT-363_SC-70-6_Handsoldering, symbol 74xGxx:74LVC1G97
- R1, R2: value R -> 10k
Connections:
- net LV is gone; now on net RPI_RXD: Q2.2 (S), R1.2
- net +5V: now also IC1.6 (E1), L1.2, Q3.3, C4.2, C5.1, C6.1, C7.1, R4.2
- net GND: now also J1.14 (GND), J1.20 (GND), J1.25 (GND), J1.30 (GND), J1.34 (GND), J1.39 (GND), J1.6 (GND), J1.9 (GND), PS1.1 (GND), C1.2, C2.2, C5.2, C6.2, C7.2, R5.1, R6.2, R7.2, U3.2 (GND)
- net RPI_RXD: no longer U1.6 (PB1)
- net VCC: now also U3.5 (VCC)
- net 5V_RPI: now reaches J1.2 (5V)
- net 5V_RPI: now also IC1.5 (E2), J1.4 (5V), Q3.2
- net at Q3.1: now also IC1.4 (C2), R7.1
- net at IC1.1 (C1): now also IC1.2 (B1), IC1.3 (B2), R6.1
- net at L1.1: now also PS1.2 (SW), C3.2
- net VIN: now reaches PS1.3 (VIN)
- net VIN: now also C1.1, C2.1, R3.2
- net at PS1.4 (FB): now also C4.1, R4.1, R5.2
- net at PS1.5 (EN): now also R3.1
- net at PS1.6 (BOOT): now also C3.1
- net HV renamed ATTINY_TX
- net ATTINY_TX: now also U1.6 (PB1)
- net RPI_TXD renamed ATTINY_RX
Other:
- moved on the sheet: IC1, J1, J2, J3, L1, PS1, Q1, Q2, Q3, R1, R2, U1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

Commit message: big save before Pico
Parts:
- removed C7: 22uF, Capacitor_SMD:C_1206_3216Metric_Pad1.33x1.80mm_HandSolder, symbol Device:CP
- added IC2: MC74HC32ADG, MC74HC32ADG:MC74HC32ADG, symbol MC74HC32ADG:MC74HC32ADG
- added J5: 39502-1003, 39502-1003:39502-1003, symbol 39502-1003:39502-1003
- added J6, J7: 39502-1002, 39502-1002:39502-1002, symbol 39502-1002:39502-1002
- added R10, R11: 10k, Resistor_SMD:R_0805_2012Metric_Pad1.20x1.40mm_HandSolder, symbol Device:R
- added R8: ?, Resistor_SMD:R_0603_1608Metric_Pad0.98x0.95mm_HandSolder, symbol Device:R
- added R9: 13.3k, Resistor_SMD:R_0603_1608Metric_Pad0.98x0.95mm_HandSolder, symbol Device:R
- added U4: SC0915, raspberry-pi-pico-r3-1:raspberry-pi-pico-r3-1, symbol raspberry-pi-pico-r3-1:SC0915
- C4: value 91pF -> 75pF
- R3: value 100k -> ?
- R4: value 100k -> 49.9k
- R5: value 13.7k -> 100k
Connections:
- net +3V3: now also Q1.1 (G), R10.1
- net +5V: now also R11.1; no longer C4.2
- net ATTINY_TX: now also Q1.3 (D), R11.2
- net GND: now also IC2.7 (GND), R8.1, R9.1, U4.13 (GND), U4.18 (GND), U4.23 (GND), U4.28 (GND), U4.3 (GND), U4.33 (AGND/GND), U4.38 (GND), U4.8 (GND), U4.A (GND), U4.B (GND), U4.C (GND), U4.D (GND), U4.D2 (GND), U4.TP1 (GND); no longer R5.1
- net RPI_RXD: now also Q1.2 (S), R10.2
- net at C4.1, R4.1, R5.2: no longer PS1.4 (FB)
- net at PS1.5 (EN), R3.1: now also R8.2
- new net: C4.2, PS1.4 (FB), R5.1, R9.2
- new net 3V3_EN: U4.37 (3V3_EN)
- new net A1: IC2.1 (A1)
- new net A4: IC2.12 (A4)
- new net B1: IC2.2 (B1)
- new net B4: IC2.13 (B4)
- new net RUN: U4.30 (RUN)
- new net SWCLK: U4.D1 (SWCLK)
- new net SWDIO: U4.D3 (SWDIO)
- new net VSYS: U4.39 (VSYS)
- new net Y1: IC2.3 (Y1)
- new net Y4: IC2.11 (Y4)
- no-connect marks 0 -> 6
Other:
- note added: "15 uH kellene ide az adatlap szerint"
- note added: "3V3 input for Pico"
- note added: "a kapcsolás nem stimmel teljesen még: https://www.ti.com/lit/ds/symlink/tps54202.pdf?ts=1676556598442&ref_url=https%253A%252F%252Fwww.ti.com%252Fproduct%252FTPS54202%252Fpart-details%252FTPS54202DDCR%253Futm_source%253Dgoogle%2526utm_medium%253Dcpc%2526utm_campaign%253Docb-tistore-promo-app_opn_en-cpc-storeic-google-wwe%2526utm_content%253DDevice%2526ds_k%253DTPS54202DDCR%2526DCM%253Dyes%2526gcli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"
- moved on the sheet: C4, C5, C6, R4, R5
